Commit message: Update mrm.xacro

File: mrm.xacro (robot description, xacro)
@@ -1,139 +1,81 @@
 <?xml version="1.0" ?>
 <robot name="mrm" xmlns:xacro="http://www.ros.org/wiki/xacro">
-    <link name="base_link">
-        <visual>
-            <origin rpy="0 0 0" xyz="0 0 0"/>
-             <material name="black">
-                <color rgba="${0/255} ${0/255} ${0/255} 1.0"/>
-            </material>
-            <geometry>
-                <box size="1.0 1.0 1.0"/>
-            </geometry>
-        </visual>
-	<collision>
-      		<geometry>
-        		<box size="1.0 1.0 1.0"/>
-      		</geometry>
-   	 </collision>
-   	 <inertial>
-     		 <mass value="100"/>
-     		 <inertia ixx="0.8333" ixy="0.0" ixz="0.0" iyy="0.8333" iyz="0.0" izz="0.8333"/>
-    	 </inertial>
-    </link>
-    <joint name="base_link__link_01" type="revolute">
-        <axis xyz="0 0 1" />
-        <limit effort="1000.0" lower="-3.14" upper="3.14" velocity="0.5" />
-        <origin rpy="0 0 0" xyz="0 0 0.5"/>
-        <parent link="base_link"/>
-        <child link="link1"/>
-    </joint>
-    <transmission name="trans_base_link__link_01">
-      <type>transmission_interface/SimpleTransmission</type>
-      <joint name="base_link__link_01">
-        <hardwareInterface>hardware_interface/EffortJointInterface</hardwareInterface>
-      </joint>
-      <actuator name="motor_base_link__link_01">
-        <hardwareInterface>hardware_interface/EffortJointInterface</hardwareInterface>
-        <mechanicalReduction>1</mechanicalReduction>
-      </actuator>
-    </transmission>
-    <link name="link1">
-        <visual>
-            <origin rpy="0 0 0" xyz="0 0 0.2"/>
-	    <material name="orange">
-                <color rgba="${255/255} ${108/255} ${10/255} 1.0"/>
-            </material>
-            <geometry>
-                <cylinder radius="0.09" length="1.2"/>
-            </geometry>
-        </visual>
-	<collision>
-      		<geometry>
-        		<cylinder length="1.2" radius="0.09"/>
-      		</geometry>
-   	 </collision>
-   	 <inertial>
-     		 <mass value="10"/>
-     		 <inertia ixx="0.12202" ixy="0.0" ixz="0.0" iyy="0.12202" iyz="0.0" izz="0.00405"/>
-    	 </inertial>
-    </link>
-<joint name="link_01__link_02" type="revolute">
-        <axis xyz="1 0 0" />
-        <limit effort="1000.0" lower="-2.45" upper="2.45" velocity="0.5" />
-        <origin rpy="0 0 0" xyz="0 0 0.8"/>
-        <parent link="link1"/>
-        <child link="link2"/>
-    </joint>
-<transmission name="trans_link_01__link_02">
-      <type>transmission_interface/SimpleTransmission</type>
-      <joint name="link_01__link_02">
-        <hardwareInterface>hardware_interface/EffortJointInterface</hardwareInterface>
-      </joint>
-      <actuator name="motor_link_01__link_01">
-        <hardwareInterface>hardware_interface/EffortJointInterface</hardwareInterface>
-        <mechanicalReduction>1</mechanicalReduction>
-      </actuator>
-    </transmission>
-    <link name="link2">
-        <visual>
-            <origin rpy="0 0 0" xyz="0 0 0.25"/>
-             <material name="white">
-                <color rgba="${255/255} ${255/255} ${255/255} 1.0"/>
-            </material>
-            <geometry>
-                <cylinder radius="0.09" length="1.2"/>
-            </geometry>
-        </visual>
-	<collision>
-      		<geometry>
-        		<cylinder length="1.2" radius="0.09"/>
-      		</geometry>
-   	 </collision>
-   	 <inertial>
-     		 <mass value="10"/>
-     		 <inertia ixx="0.12202" ixy="0.0" ixz="0.0" iyy="0.12202" iyz="0.0" izz="0.00405"/>
-    	 </inertial>
-    </link>
-<joint name="link_02__link_03" type="revolute">
-        <axis xyz="1 0 0" />
-        <limit effort="1000.0" lower="-2.45" upper="2.45" velocity="0.5" />
-        <origin rpy="0 0 0" xyz="0 0 0.8"/>
-        <parent link="link2"/>
-        <child link="link3"/>
-    </joint>
-<transmission name="trans_link_02__link_03">
-      <type>transmission_interface/SimpleTransmission</type>
-      <joint name="link_02__link_03">
-        <hardwareInterface>hardware_interface/EffortJointInterface</hardwareInterface>
-      </joint>
-      <actuator name="motor_link_02__link_03">
-        <hardwareInterface>hardware_interface/EffortJointInterface</hardwareInterface>
-        <mechanicalReduction>1</mechanicalReduction>
-      </actuator>
-    </transmission>
-    <link name="link3">
-        <visual>
-            <origin rpy="0 0 0" xyz="0 0 0.25"/>
-             <material name="orange">
-                <color rgba="${255/255} ${108/255} ${10/255} 1.0"/>
-            </material>
-            <geometry>
-                <cylinder radius="0.09" length="1.2"/>
-            </geometry>
-        </visual>
- 	<collision>
-      		<geometry>
-        		<cylinder length="1.2" radius="0.09"/>
-      		</geometry>
-   	 </collision>
-   	 <inertial>
-     		 <mass value="10"/>
-     		 <inertia ixx="0.12202" ixy="0.0" ixz="0.0" iyy="0.12202" iyz="0.0" izz="0.00405"/>
-    	 </inertial>
-    </link>
-<gazebo>
+  <!-- BGN - Include -->
+  <xacro:include filename="$(find mrm_description)/urdf/robot_parameters.xacro" />
+  <xacro:include filename="$(find mrm_description)/urdf/links_joints.xacro" />
+  <!-- END - Include -->
+  <!-- BGN - Robot description -->
+  <m_link_box name="${link_00_name}"
+              origin_rpy="0 0 0" origin_xyz="0 0 0"
+              mass="1024"
+              ixx="170.667" ixy="0" ixz="0"
+              iyy="170.667" iyz="0"
+              izz="170.667"
+              size="1 1 1" />
+  <m_joint name="${link_00_name}__${link_01_name}" type="revolute"
+           axis_xyz="0 0 1"
+           origin_rpy="0 0 0" origin_xyz="0 0 0.5"
+           parent="base_link" child="link_01"
+           limit_e="1000" limit_l="-3.14" limit_u="3.14" limit_v="0.5" />
+  <m_link_mesh name="${link_01_name}"
+              origin_rpy="0 0 0" origin_xyz="0 0 -0.1"
+              mass="157.633"
+              ixx="13.235" ixy="0" ixz="0"
+              iyy="13.235" iyz="0"
+              izz="9.655"
+              meshfile="package://mrm_description/meshes/Link1-v2.stl"
+              meshscale="0.001 0.001 0.001" />
+  <m_joint name="${link_01_name}__${link_02_name}" type="revolute"
+           axis_xyz="0 1 0"
+           origin_rpy="0 0 0" origin_xyz="0 0 0.4"
+           parent="link_01" child="link_02"
+           limit_e="1000" limit_l="0" limit_u="0.5" limit_v="0.5" />
+  <m_link_cylinder name="${link_02_name}"
+              origin_rpy="0 0 0" origin_xyz="0 0 0.4"
+              mass="57.906"
+              ixx="12.679" ixy="0" ixz="0"
+              iyy="12.679" iyz="0"
+              izz="0.651"
+              radius="0.15" length="0.8" />
+  <m_joint name="${link_02_name}__${link_03_name}" type="revolute"
+           axis_xyz="0 1 0"
+           origin_rpy="0 0 0" origin_xyz="0 0 0.8"
+           parent="link_02" child="link_03"
+           limit_e="1000" limit_l="0" limit_u="0.75" limit_v="0.5" />
+  <m_link_cylinder name="${link_03_name}"
+              origin_rpy="0 0 0" origin_xyz="0 0 0.4"
+              mass="57.906"
+              ixx="12.679" ixy="0" ixz="0"
+              iyy="12.679" iyz="0"
+              izz="0.651"
+              radius="0.15" length="0.8" />
+  <m_joint name="${link_03_name}__${link_04_name}" type="revolute"
+           axis_xyz="0 1 0"
+           origin_rpy="0 0 0" origin_xyz="0 0 0.8"
+           parent="link_03" child="link_04"
+           limit_e="1000" limit_l="0" limit_u="0.75" limit_v="0.5" />
+  <m_link_cylinder name="${link_04_name}"
+              origin_rpy="0 0 0" origin_xyz="0 0 0.4"
+              mass="57.906"
+              ixx="12.679" ixy="0" ixz="0"
+              iyy="12.679" iyz="0"
+              izz="0.651"
+              radius="0.15" length="0.8" />
+  <m_joint name="${link_04_name}__${link_05_name}" type="revolute"
+           axis_xyz="0 0 1"
+           origin_rpy="0 0 0" origin_xyz="0 0 0.8"
+           parent="link_04" child="link_05"
+           limit_e="1000" limit_l="-3.14" limit_u="3.14" limit_v="0.5" />
+  <m_link_cylinder name="${link_05_name}"
+              origin_rpy="0 0 0" origin_xyz="0 0 0.125"
+              mass="18.056"
+              ixx="0.479" ixy="0" ixz="0"
+              iyy="0.479" iyz="0"
+              izz="0.204"
+              radius="0.15" length="0.25" />
+  <!-- END - Robot description
+  <gazebo>
     <plugin name="gazebo_ros_control" filename="libgazebo_ros_control.so">
-    <robotNamespace>/robotarm</robotNamespace>
     </plugin>
-</gazebo>
+  </gazebo>
 </robot>
